Commit message: remove <inertia> tag, update package name to "snake_description"

File: urdf/snake_tool.urdf (robot description, URDF)
Before this commit: robot snake_tool, 29 links, 28 joints
Links:
- link link_00: mass 0.000527534386374249 -> None; geometry collision mesh filename=package://snake_description/meshes/link_00.STL scale=0.001 0.001 0.001; visual mesh filename=package://snake_description/meshes/link_00.STL scale=0.001 0.001 0.001
- link link_01: mass 1.27452758455881E-05 -> None; geometry collision mesh filename=package://snake_description/meshes/link_01.STL scale=0.001 0.001 0.001; visual mesh filename=package://snake_description/meshes/link_01.STL scale=0.001 0.001 0.001
- link link_02: mass 1.25940330913542E-05 -> None; geometry collision mesh filename=package://snake_description/meshes/link_02.STL scale=0.001 0.001 0.001; visual mesh filename=package://snake_description/meshes/link_02.STL scale=0.001 0.001 0.001
- link link_03: mass 1.24583333094806E-05 -> None; geometry collision mesh filename=package://snake_description/meshes/link_03.STL scale=0.001 0.001 0.001; visual mesh filename=package://snake_description/meshes/link_03.STL scale=0.001 0.001 0.001
- link link_04: mass 1.23074072610594E-05 -> None; geometry collision mesh filename=package://snake_description/meshes/link_04.STL scale=0.001 0.001 0.001; visual mesh filename=package://snake_description/meshes/link_04.STL scale=0.001 0.001 0.001
- link link_05: mass 1.21725767298699E-05 -> None; geometry collision mesh filename=package://snake_description/meshes/link_05.STL scale=0.001 0.001 0.001; visual mesh filename=package://snake_description/meshes/link_05.STL scale=0.001 0.001 0.001
- link link_06: mass 1.20222329033018E-05 -> None; geometry collision mesh filename=package://snake_description/meshes/link_06.STL scale=0.001 0.001 0.001; visual mesh filename=package://snake_description/meshes/link_06.STL scale=0.001 0.001 0.001
- link link_07: mass 1.16358994606626E-05 -> None; geometry collision mesh filename=package://snake_description/meshes/link_07.STL scale=0.001 0.001 0.001; visual mesh filename=package://snake_description/meshes/link_07.STL scale=0.001 0.001 0.001
- link link_08: mass 1.14861453684126E-05 -> None; geometry collision mesh filename=package://snake_description/meshes/link_08.STL scale=0.001 0.001 0.001; visual mesh filename=package://snake_description/meshes/link_08.STL scale=0.001 0.001 0.001
- link link_09: mass 1.16046349573238E-05 -> None; geometry collision mesh filename=package://snake_description/meshes/link_09.STL scale=0.001 0.001 0.001; visual mesh filename=package://snake_description/meshes/link_09.STL scale=0.001 0.001 0.001
- link link_10: mass 1.14554812323596E-05 -> None; geometry collision mesh filename=package://snake_description/meshes/link_10.STL scale=0.001 0.001 0.001; visual mesh filename=package://snake_description/meshes/link_10.STL scale=0.001 0.001 0.001
- link link_11: mass 1.1322448006399E-05 -> None; geometry collision mesh filename=package://snake_description/meshes/link_11.STL scale=0.001 0.001 0.001; visual mesh filename=package://snake_description/meshes/link_11.STL scale=0.001 0.001 0.001
- link link_12: mass 1.11738855922553E-05 -> None; geometry collision mesh filename=package://snake_description/meshes/link_12.STL scale=0.001 0.001 0.001; visual mesh filename=package://snake_description/meshes/link_12.STL scale=0.001 0.001 0.001
- link link_13: mass 1.10414439583088E-05 -> None; geometry collision mesh filename=package://snake_description/meshes/link_13.STL scale=0.001 0.001 0.001; visual mesh filename=package://snake_description/meshes/link_13.STL scale=0.001 0.001 0.001
- link link_14: mass 1.08934757683148E-05 -> None; geometry collision mesh filename=package://snake_description/meshes/link_14.STL scale=0.001 0.001 0.001; visual mesh filename=package://snake_description/meshes/link_14.STL scale=0.001 0.001 0.001
- link link_15: mass 1.07631201406372E-05 -> None; geometry collision mesh filename=package://snake_description/meshes/link_15.STL scale=0.001 0.001 0.001; visual mesh filename=package://snake_description/meshes/link_15.STL scale=0.001 0.001 0.001
- link link_16: mass 1.05164541743147E-05 -> None; geometry collision mesh filename=package://snake_description/meshes/link_16.STL scale=0.001 0.001 0.001; visual mesh filename=package://snake_description/meshes/link_16.STL scale=0.001 0.001 0.001
- link link_17: mass 1.02334472879023E-05 -> None; geometry collision mesh filename=package://snake_description/meshes/link_17.STL scale=0.001 0.001 0.001; visual mesh filename=package://snake_description/meshes/link_17.STL scale=0.001 0.001 0.001
- link link_18: mass 1.00854062599699E-05 -> None; geometry collision mesh filename=package://snake_description/meshes/link_18.STL scale=0.001 0.001 0.001; visual mesh filename=package://snake_description/meshes/link_18.STL scale=0.001 0.001 0.001
- link link_19: mass 1.02078004597305E-05 -> None; geometry collision mesh filename=package://snake_description/meshes/link_19.STL scale=0.001 0.001 0.001; visual mesh filename=package://snake_description/meshes/link_19.STL scale=0.001 0.001 0.001
- link link_20: mass 1.00605032731873E-05 -> None; geometry collision mesh filename=package://snake_description/meshes/link_20.STL scale=0.001 0.001 0.001; visual mesh filename=package://snake_description/meshes/link_20.STL scale=0.001 0.001 0.001
- link link_21: mass 9.95419229086504E-06 -> None; geometry collision mesh filename=package://snake_description/meshes/link_21.STL scale=0.001 0.001 0.001; visual mesh filename=package://snake_description/meshes/link_21.STL scale=0.001 0.001 0.001
- link link_22: mass 9.89934772982008E-06 -> None; geometry collision mesh filename=package://snake_description/meshes/link_22.STL scale=0.001 0.001 0.001; visual mesh filename=package://snake_description/meshes/link_22.STL scale=0.001 0.001 0.001
- link link_23: mass 9.90814006667915E-06 -> None; geometry collision mesh filename=package://snake_description/meshes/link_23.STL scale=0.001 0.001 0.001; visual mesh filename=package://snake_description/meshes/link_23.STL scale=0.001 0.001 0.001
- link link_24: mass 9.89934772981781E-06 -> None; geometry collision mesh filename=package://snake_description/meshes/link_24.STL scale=0.001 0.001 0.001; visual mesh filename=package://snake_description/meshes/link_24.STL scale=0.001 0.001 0.001
- link link_25: mass 9.90814006668526E-06 -> None; geometry collision mesh filename=package://snake_description/meshes/link_25.STL scale=0.001 0.001 0.001; visual mesh filename=package://snake_description/meshes/link_25.STL scale=0.001 0.001 0.001
- link link_26: mass 9.89934772981985E-06 -> None; geometry collision mesh filename=package://snake_description/meshes/link_26.STL scale=0.001 0.001 0.001; visual mesh filename=package://snake_description/meshes/link_26.STL scale=0.001 0.001 0.001
- link link_27: mass 2.79672420357717E-05 -> None; geometry collision mesh filename=package://snake_description/meshes/link_27.STL scale=0.001 0.001 0.001; visual mesh filename=package://snake_description/meshes/link_27.STL scale=0.001 0.001 0.001
- link link_ee: mass 2.79672420357717E-05 -> None; geometry 

Commit message: adjust joint limits

File: urdf/snake_tool.urdf (robot description, URDF)
Before this commit: robot snake_tool, 29 links, 28 joints
Joints:
- joint joint_00: limit lower=0 upper=0 effort=0 velocity=0 -> lower=-0.16 upper=0.16 effort=0 velocity=0
- joint joint_01: limit lower=0 upper=0 effort=0 velocity=0 -> lower=-0.16 upper=0.16 effort=0 velocity=0
- joint joint_02: limit lower=0 upper=0 effort=0 velocity=0 -> lower=-0.16 upper=0.16 effort=0 velocity=0
- joint joint_03: limit lower=0 upper=0 effort=0 velocity=0 -> lower=-0.16 upper=0.16 effort=0 velocity=0
- joint joint_04: limit lower=0 upper=0 effort=0 velocity=0 -> lower=-0.16 upper=0.16 effort=0 velocity=0
- joint joint_06: limit lower=0 upper=0 effort=0 velocity=0 -> lower=-0.16 upper=0.16 effort=0 velocity=0
- joint joint_07: limit lower=0 upper=0 effort=0 velocity=0 -> lower=-0.16 upper=0.16 effort=0 velocity=0
- joint joint_08: limit lower=0 upper=0 effort=0 velocity=0 -> lower=-0.16 upper=0.16 effort=0 velocity=0
- joint joint_09: limit lower=0 upper=0 effort=0 velocity=0 -> lower=-0.16 upper=0.16 effort=0 velocity=0
- joint joint_10: limit lower=0 upper=0 effort=0 velocity=0 -> lower=-0.16 upper=0.16 effort=0 velocity=0
- joint joint_11: limit lower=0 upper=0 effort=0 velocity=0 -> lower=-0.16 upper=0.16 effort=0 velocity=0
- joint joint_12: limit lower=0 upper=0 effort=0 velocity=0 -> lower=-0.16 upper=0.16 effort=0 velocity=0
- joint joint_13: limit lower=0 upper=0 effort=0 velocity=0 -> lower=-0.16 upper=0.16 effort=0 velocity=0
- joint joint_14: limit lower=0 upper=0 effort=0 velocity=0 -> lower=-0.16 upper=0.16 effort=0 velocity=0
- joint joint_15: limit lower=0 upper=0 effort=0 velocity=0 -> lower=-0.16 upper=0.16 effort=0 velocity=0
- joint joint_16: limit lower=0 upper=0 effort=0 velocity=0 -> lower=-0.16 upper=0.16 effort=0 velocity=0
- joint joint_17: limit lower=0 upper=0 effort=0 velocity=0 -> lower=-0.16 upper=0.16 effort=0 velocity=0
- joint joint_18: limit lower=0 upper=0 effort=0 velocity=0 -> lower=-0.16 upper=0.16 effort=0 velocity=0
- joint joint_19: limit lower=0 upper=0 effort=0 velocity=0 -> lower=-0.16 upper=0.16 effort=0 velocity=0
- joint joint_20: limit lower=0 upper=0 effort=0 velocity=0 -> lower=-0.16 upper=0.16 effort=0 velocity=0
- joint joint_21: limit lower=0 upper=0 effort=0 velocity=0 -> lower=-0.16 upper=0.16 effort=0 velocity=0
- joint joint_22: limit lower=0 upper=0 effort=0 velocity=0 -> lower=-0.16 upper=0.16 effort=0 velocity=0
- joint joint_23: limit lower=0 upper=0 effort=0 velocity=0 -> lower=-0.16 upper=0.16 effort=0 velocity=0
- joint joint_24: limit lower=0 upper=0 effort=0 velocity=0 -> lower=-0.16 upper=0.16 effort=0 velocity=0
- joint joint_25: limit lower=0 upper=0 effort=0 velocity=0 -> lower=-0.16 upper=0.16 effort=0 velocity=0
- joint joint_26: limit lower=0 upper=0 effort=0 velocity=0 -> lower=-0.16 upper=0.16 effort=0 velocity=0
